File: pannel108-withdems.kicad_pcb (KiCad board)
At the start: 2 copper layers, 108 x 108 mm, 32 parts

Commit message: updates
Parts:
- moved REF** 123.9 mm to (195.6, 98.5)
- moved REF** 123.9 mm to (278.1, 98.5)
- moved REF** 123.7 mm to (195.6, 30.5)
- moved REF** 123.7 mm to (278.1, 30.5)
Other:
- board text removed: "108mm x 180mm Pannel"
