File: pannel108-v2.kicad_pcb (KiCad board)
At the start: 2 copper layers, 107.9 x 107.9 mm, 32 parts

Commit message: updates
Other:
- board text added: "108mm x 108mm Sub Fixation Panel"
- board text removed: "108mm x 180mm Panel use 25mills (0.6350mm)"
