File: pannel_subboard.kicad_pcb (KiCad board)
At the start: 2 copper layers, 90.2 x 76.2 mm, 32 parts, among them J1 Conn_01x02, J10 Conn_02x14_Counter_Clockwise, J2 Conn_01x05, J3 Conn_01x05, J4 Conn_01x05, J5 Conn_01x05, J6 Conn_01x05, J7 Conn_01x05, J8 Conn_01x05, J9 Conn_01x05

Commit message: updates
Parts:
- added J11: Conn_01x05, Pin_Headers:Pin_Header_Straight_1x05_Pitch2.54mm, F.Cu at (76.8, 74.3)
- added J12: Conn_01x05, Pin_Headers:Pin_Header_Straight_1x05_Pitch2.54mm, F.Cu at (122.6, 74.3)
- added J13: Conn_01x05, Pin_Headers:Pin_Header_Straight_1x05_Pitch2.54mm, F.Cu at (76.8, 107.4)
- added J14: Conn_01x05, Pin_Headers:Pin_Header_Straight_1x05_Pitch2.54mm, F.Cu at (122.6, 107.4)
- added J15: Conn_01x05, Pin_Headers:Pin_Header_Straight_1x05_Pitch2.54mm, F.Cu at (99.7, 74.3)
- added J16: Conn_01x05, Pin_Headers:Pin_Header_Straight_1x05_Pitch2.54mm, F.Cu at (145.4, 74.3)
- added J17: Conn_01x05, Pin_Headers:Pin_Header_Straight_1x05_Pitch2.54mm, F.Cu at (99.7, 107.4)
- added J18: Conn_01x05, Pin_Headers:Pin_Header_Straight_1x05_Pitch2.54mm, F.Cu at (145.4, 107.4)
- moved J1 0.64 mm to (90.2, 60.4)
- moved D1 0.63 mm to (83.2, 62.9)
- moved R1 0.63 mm to (87.0, 61.0)
Routing:
- net SW8-A: track 71.0 -> 90.7 mm
- net SW8-B: track 71.3 -> 91.0 mm
- net SW8-C: track 72.1 -> 91.8 mm
- net SW4-B: track 45.4 -> 61.0 mm, vias 0 -> 1
- net SW7-A: track 59.4 -> 74.4 mm
- net SW5-C: track 61.0 -> 74.8 mm
- net SW7-B: track 62.7 -> 76.2 mm
- net SW5-B: track 56.8 -> 70.2 mm
- net SW1-C: track 24.8 -> 38.2 mm
- net SW1-B: track 21.2 -> 34.6 mm
- net SW6-A: track 54.8 -> 67.5 mm
- net SW5-A: track 53.2 -> 65.9 mm
- net SW2-C: track 22.6 -> 35.3 mm
- net SW1-A: track 17.7 -> 30.4 mm
- net SW6-C: track 57.9 -> 70.6 mm
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Other:
- board text added: "GND"
- board text added: "VCC"
