File: pannel108-cleanoverlay-v2.kicad_pcb (KiCad board)
At the start: 2 copper layers, 107.9 x 107.9 mm, 12 parts

Commit message: updates
Other:
- board text added: "108mm x 108mm Overlay Panel"
- board text removed: "108mm x 180mm Panel use 25mills (0.6350mm)"
Changed lines of the file:
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@@
   (gr_line (start 63.5 149.91) (end 171.45 41.96) (layer Dwgs.User) (width 0.15))
   (gr_line (start 63.5 41.96) (end 171.45 149.91) (layer Dwgs.User) (width 0.15))
-  (gr_text "108mm x 180mm Panel\nuse 25mills (0.6350mm)" (at 118.745 141.02) (layer F.SilkS)
+  (gr_text "108mm x 108mm Overlay Panel" (at 118.745 141.02) (layer F.SilkS)
     (effects (font (size 1.5 1.5) (thickness 0.2)))
   )
