File: pannel_subboard.sch (KiCad schematic (older format))
At the start: 12 parts, among them J1 Conn_01x02, J10 Conn_02x14_Counter_Clockwise, J2 Conn_01x05, J3 Conn_01x05, J4 Conn_01x05, J5 Conn_01x05, J6 Conn_01x05, J7 Conn_01x05, J8 Conn_01x05, J9 Conn_01x05

Commit message: updates
Parts:
- added J11, J12, J13, J14, J15, J16, J17, J18: Conn_01x05, Pin_Headers:Pin_Header_Straight_1x05_Pitch2.54mm, symbol Connector_Generic:Conn_01x05
Connections:
- net GND: now also J11.5 (Pin_5), J12.5 (Pin_5), J13.5 (Pin_5), J14.5 (Pin_5), J15.5 (Pin_5), J16.5 (Pin_5), J17.5 (Pin_5), J18.5 (Pin_5)
- net SW1-A: now also J11.2 (Pin_2)
- net SW1-B: now also J11.3 (Pin_3)
- net SW1-C: now also J11.4 (Pin_4)
- net SW2-A: now also J15.2 (Pin_2)
- net SW2-B: now also J15.3 (Pin_3)
- net SW2-C: now also J15.4 (Pin_4)
- net SW3-A: now also J12.2 (Pin_2)
- net SW3-B: now also J12.3 (Pin_3)
- net SW3-C: now also J12.4 (Pin_4)
- net SW4-A: now also J16.2 (Pin_2)
- net SW4-B: now also J16.3 (Pin_3)
- net SW4-C: now also J16.4 (Pin_4)
- net SW5-A: now also J13.2 (Pin_2)
- net SW5-B: now also J13.3 (Pin_3)
- net SW5-C: now also J13.4 (Pin_4)
- net SW6-A: now also J17.2 (Pin_2)
- net SW6-B: now also J17.3 (Pin_3)
- net SW6-C: now also J17.4 (Pin_4)
- net SW7-A: now also J14.2 (Pin_2)
- net SW7-B: now also J14.3 (Pin_3)
- net SW7-C: now also J14.4 (Pin_4)
- net SW8-A: now also J18.2 (Pin_2)
- net SW8-B: now also J18.3 (Pin_3)
- net SW8-C: now also J18.4 (Pin_4)
- net VCC: now also J11.1 (Pin_1), J12.1 (Pin_1), J13.1 (Pin_1), J14.1 (Pin_1), J15.1 (Pin_1), J16.1 (Pin_1), J17.1 (Pin_1), J18.1 (Pin_1)
Other:
- moved on the sheet: J10, J2, J3, J4, J5, J6, J7, J8, J9

Commit message: updates
Parts:
- added C?: C, symbol Device:C
- added R? (x2): R, symbol Device:R
- added SW?: SW_DPST, symbol Switch:SW_DPST
Connections:
- net GND: now also C?.2, SW?.2, SW?.4
- net VCC: now also R?.2
- new net EXT_A: R?.1, R?.2, SW?.1, SW?.3
- new net OUT: C?.1, R?.1
Changed lines of the file:
@@
 Text GLabel 3200 5350 0    50   Input ~ 0
 SW8-C
+$Comp
+L Device:R R?
+U 1 1 618725A2
+P 1200 6600
+F 0 "R?" H 1270 6646 50  0000 L CNN
+F 1 "R" H 1270 6555 50  0000 L CNN
+F 2 "" V 1130 6600 50  0001 C CNN
+F 3 "~" H 1200 6600 50  0001 C CNN
+	1    1200 6600
+	1    0    0    -1
+$EndComp
+$Comp
+L Device:C C?
+U 1 1 61874002
+P 2150 6600
+F 0 "C?" H 2265 6646 50  0000 L CNN
+F 1 "C" H 2265 6555 50  0000 L CNN
+F 2 "" H 2188 6450 50  0001 C CNN
+F 3 "~" H 2150 6600 50  0001 C CNN
+	1    2150 6600
+	1    0    0    -1
+$EndComp
+$Comp
+L Switch:SW_DPST SW?
+U 1 1 618764A4
+P 1700 6950
+F 0 "SW?" H 1700 7275 50  0000 C CNN
+F 1 "SW_DPST" H 1700 7184 50  0000 C CNN
+F 2 "" H 1700 6950 50  0001 C CNN
+F 3 "~" H 1700 6950 50  0001 C CNN
+	1    1700 6950
+	1    0    0    -1
+$EndComp
+$Comp
+L power:GND #PWR?
+U 1 1 61877420
+P 2150 7300
+F 0 "#PWR?" H 2150 7050 50  0001 C CNN
+F 1 "GND" V 2155 7172 50  0000 R CNN
+F 2 "" H 2150 7300 50  0001 C CNN
+F 3 "" H 2150 7300 50  0001 C CNN
+	1    2150 7300
+	1    0    0    -1
+$EndComp
+$Comp
+L power:VCC #PWR?
+U 1 1 6187796B
+P 1200 7350
+F 0 "#PWR?" H 1200 7200 50  0001 C CNN
+F 1 "VCC" V 1215 7477 50  0000 L CNN
+F 2 "" H 1200 7350 50  0001 C CNN
+F 3 "" H 1200 7350 50  0001 C CNN
+	1    1200 7350
+	-1   0    0    1
+$EndComp
+$Comp
+L Device:R R?
+U 1 1 618762FB
+P 1200 7200
+F 0 "R?" H 1270 7246 50  0000 L CNN
+F 1 "R" H 1270 7155 50  0000 L CNN
+F 2 "" V 1130 7200 50  0001 C CNN
+F 3 "~" H 1200 7200 50  0001 C CNN
+	1    1200 7200
+	1    0    0    -1
+$EndComp
+Wire Wire Line
+	1200 7050 1200 6850
+Wire Wire Line
+	2150 6850 1900 6850
+Wire Wire Line
+	2150 6750 2150 6850
+Wire Wire Line
+	2150 6850 2150 7300
+Connection ~ 2150 6850
+Wire Wire Line
+	1900 7050 1900 7250
+Wire Wire Line
+	1500 7050 1500 7250
+Wire Wire Line
+	1200 6850 1200 6750
+Connection ~ 1200 6850
+Wire Wire Line
+	1200 6350 1200 6450
+Wire Wire Line
+	2150 6350 2150 6450
+Text GLabel 1650 6250 1    50   Input ~ 0
+OUT
+Wire Wire Line
+	1500 6850 1200 6850
+Wire Wire Line
+	1200 6350 1650 6350
+Wire Wire Line
+	1500 7050 1500 6850
+Connection ~ 1500 7050
+Connection ~ 1500 6850
+Wire Wire Line
+	1900 7050 1900 6850
+Connection ~ 1900 7050
+Connection ~ 1900 6850
+Text GLabel 1500 7250 3    50   Input ~ 0
+EXT_A
+Text GLabel 1900 7250 3    50   Input ~ 0
+EXT_B
+Wire Wire Line
+	1650 6250 1650 6350
+Connection ~ 1650 6350
+Wire Wire Line
+	1650 6350 2150 6350
 $EndSCHEMATC
